File: GitHub Projects/CRAP Project/Flight Controller.sch (EAGLE design)
At the start: 1 part

Commit message: Added Screw Terminals and Schematic Frames
Added screw in terminals of the 2, 4, and 8 widths.  They are at a
2.54mm pitch (0.1').
Also added in schematic frames to make our things look much fancier.
Other:
- note removed: "Accelerometer(s) Sheet"
- note removed: "Power Design Sheet"
- note removed: "Tempurature Sensing Sheet"
Changed lines of the file:
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@@
 <?xml version="1.0" encoding="utf-8"?>
 <!DOCTYPE eagle SYSTEM "eagle.dtd">
-<eagle version="8.0.1">
+<eagle version="8.0.0">
 <drawing>
 <settings>
@@
 </classes>
 <modules>
-<module name="MS5611" prefix="M" dx="30.48" dy="20.32">
+<module name="MS5611" prefix="M" dx="30.48" dy="15.24">
 <ports>
 <port name="SCLK" side="left" coord="5.08" direction="in"/>
@@
 <part name="GND1" library="supply1" deviceset="GND" device=""/>
 <part name="+3V1" library="supply1" deviceset="+3V3" device=""/>
+<part name="FRAME1" library="frames" deviceset="A3L-LOC" device=""/>
 </parts>
 <sheets>
@@
 <instance part="GND1" gate="1" x="-38.1" y="-10.16"/>
 <instance part="+3V1" gate="G$1" x="-38.1" y="7.62"/>
+<instance part="FRAME1" gate="G$1" x="-205.74" y="-129.54"/>
 </instances>
 <busses>
@@
 <part name="C10" library="rcl" deviceset="C-EU" device="C0805" value="22u"/>
 <part name="C11" library="rcl" deviceset="C-EU" device="C0805" value="22u"/>
+<part name="FRAME1" library="frames" deviceset="A3L-LOC" device=""/>
 </parts>
 <sheets>
@@
 <instance part="C10" gate="G$1" x="101.6" y="7.62"/>
 <instance part="C11" gate="G$1" x="109.22" y="7.62"/>
+<instance part="FRAME1" gate="G$1" x="-213.36" y="-121.92"/>
 </instances>
 <busses>
@@
 </variantdefs>
 <parts>
+<part name="FRAME1" library="frames" deviceset="A3L-LOC" device=""/>
 </parts>
 <sheets>
@@
 </plain>
 <instances>
+<instance part="FRAME1" gate="G$1" x="0" y="0"/>
 </instances>
 <busses>
@@
 <part name="R4" library="resistor" deviceset="R-US_" device="R0603" value="10k"/>
 <part name="C4" library="rcl" deviceset="C-EU" device="C0603" value="1u"/>
+<part name="FRAME1" library="frames" deviceset="A3L-LOC" device=""/>
 </parts>
 <sheets>
@@
 </instance>
 <instance part="C4" gate="G$1" x="30.48" y="-15.24"/>
+<instance part="FRAME1" gate="G$1" x="-180.34" y="-111.76"/>
 </instances>
 <busses>
@@
 <part name="R7" library="rcl" deviceset="R-US_" device="R0603" value="15k"/>
 <part name="C4" library="rcl" deviceset="C-EU" device="C0603" value="1u"/>
+<part name="FRAME1" library="frames" deviceset="A3L-LOC" device=""/>
 </parts>
 <sheets>
@@
 </instance>
 <instance part="C4" gate="G$1" x="99.06" y="-30.48"/>
+<instance part="FRAME1" gate="G$1" x="-104.14" y="-129.54"/>
 </instances>
 <busses>
@@
 </nets>
 </sheet>
-<sheet>
-<plain>
-<text x="0" y="2.54" size="1.778" layer="91">Power Design Sheet</text>
-</plain>
-<instances>
-</instances>
-<busses>
-</busses>
-<nets>
-</nets>
-</sheet>
-<sheet>
-<plain>
-<text x="0" y="2.54" size="1.778" layer="91">Accelerometer(s) Sheet</text>
-</plain>
-<instances>
-</instances>
-<busses>
-</busses>
-<nets>
-</nets>
-</sheet>
-<sheet>
-<plain>
-<text x="0" y="2.54" size="1.778" layer="91">Tempurature Sensing Sheet</text>
-</plain>
-<instances>
-</instances>
-<busses>
-</busses>
-<nets>
-</nets>
-</sheet>

Commit message: RTD module nearly done
1. RTD module is nearly done. Just need to figure out the connections in
and out of modules, especially for the serial data lines and power.
2. Touched up power and ordnance modules to include the correct ground
symbols.
Note: All this was done with the Eagle 7.x version files
Other:
- note added: "Header connections are not inside this module on purpose"
- note added: "J1"
- note added: "LTC3225"
- note added: "NOTE TO ROUTER: Put the following silkscreen text next to each pin: 4: EXC+ 3: S+ 2: S– 1: EXC–"
- note added: "NOTE TO THE ROUTER: Wire these as Kelvin connections where the REFIN pins are the sensing terminals!"
- note added: "Ordnance Charging and Pyro Chain Connections Cooper Barry"
- note added: "RTD Sensing Circuit Cooper Barry"
- note added: "The 10 M resistor is for fault detection if one of the RTD wires breaks."
- note added: "Why 3 resistors in parallel? A 400R resistor is not cheap, and 1.2k is a standard value in the E12 series. Also, the accuracy of the temperature is dependent on the accuracy of this set resistor, and 3 in parallel reduces the tolerance by 3x."
- note removed: "1.8V Reference"
- note removed: "10.6 Hz LPF"
- note removed: "Need a 4 pin header for each external 4-wire RTD"
- note removed: "Still need to decide which symbol to use for the local ground."
- note removed: "Still to add: Headers for battery connections"
- note removed: "To ADCs"

Commit message: Started ordnance board
Other:
- note added: "!CONT_EN Continuity Enable command"
- note added: "CONT_STAT Continuity Status"
- note added: "FIRE1"
- note added: "FIRE2"
- note added: "Ordnance connections outside of the firing chain, so we can use more than a 2-terminal block."
- note added: "Power in after diode array from super capacitors"

Commit message: Added SAMG55 and AVR and SAM JTAG headers
Created AVR JTAG headers for possible future use and also created SAM
JTAG headers for immediate use.
Added G55 into the root sheet and added recommended decoupling
capacitors to VDDIO, VDDOUT, and VDDCORE.
Parts:
- added C1: 4.7u, rcl:C-EUC0603
- added C2: 1u, rcl:C-EUC0603
- added C3: 100n, rcl:C-EUC0603
- added U1: (no value), atmel:ATSAMG55J19
- JP1: device pinhead:PINHD-2X3 -> atmel:AVR_JTAG
Connections:
- removed net X_PDI_DATA: JP1.6
- removed net X_RESET_PDI_CLK: JP1.2
- new net !SHDN: U1.SHDN
- new net CS: U1.CSB@1, U1.CSB@2
- new net MISO: U1.SDO
- new net MOSI: U1.SDI/SDA
- new net N$1: C1.1, C2.1, C3.1, JP1.GND@1, U1.C+, U1.PB6/TMS
- new net N$10: U1.CX
- new net N$2: C2.1, C2.2, JP1.VCC, U1.C-, U1.PB7/TCK
- new net N$3: C1.1, C3.1, JP1./RESET, U1.PB5/TDO, U1.VIN
- new net N$4: JP1.(TRST), U1.PB4/TDI
- new net N$5: JP1.GND@2, U1.RESET, U1.VSEL
- new net N$6: C2.2, C3.1, C3.2, U1.PROG, U1.VDDCORE, U1.VDDCORE@1, U1.VDDOUT
- new net N$7: C3.2
- new net N$8: U1.PGOOD
- new net ORD_PWR: U1.COUT
- new net SCLK: U1.SCLK
- net +3V3: now also C1.1, JP1.TCK, U1.VDD, U1.VDDIO, U1.VDDIO@1, U1.VDDIO@2, U1.VDDIO@3, U1.VDDIO@4; no longer JP1.5
- net GND: now also C1.2, C2.1, C2.2, C3.1, C3.2, JP1.TDI, JP1.TDO, JP1.TMS, U1.GND, U1.GND@1, U1.GND@2, U1.PS; no longer JP1.1
Other:
- note added: "1"
- note added: "Created by members of the CRAP team Space Hardware Club"

Commit message: Fixed the board consistency by making a new board
Do not modify the schematic unless the schematic and board are
consistant.  The easiest way to do this is to just have the board open
when you open the schematic.  This is why it asks if you want to open
both when you first open the program.

Also added a fancy logo to the Atmel chip's footprint, also found an
existing part for the Xbee900 Pro, so I added that into the schematic
and made a module for it.

Also added in modules for the memory and GPS.  That will be what I work
on next.

Outstanding things:  I think the power module is a little funky with the
ports you have on there, Cooper. Are the two return lines not a common
ground?  Why separate them?  Also I recommend changing the ports on the
module to reflect any new net name changes, as well as having a
consistent direction of the pin, so set them to "pwr" when you create
them.  This will come in handy later with design rule checks, because
it'll flag any inconsistancies.
Parts:
- added U$1: 2POS_SCREWTERM, CRAP Parts:2POS_SCREWTERM
Connections:
- new net 3V3_OUT: U$1.VOUT@1, U$1.VOUT@2
- new net N$11: U$1.EN, U$1.FORCE+, U$1.PS/SYNC
- new net N$12: U$1.SCLK
- new net N$13: U$1.SDI
- new net N$14: U$1.!DRDY
- new net N$9: U$1.P$2, U$1.PG, U$1.SDO
- new net VCC_IN: U$1.P$1
- new net VDDOUT: C2.2, C3.2, U1.VDDCORE, U1.VDDCORE@1, U1.VDDOUT
- net +3V3: now also C2.1
- net GND: now also U$1.DGND, U$1.EP, U$1.FORCE2, U$1.GND, U$1.GND@1, U$1.GND@2, U$1.PGND
- net N$1: now also U$1.BIAS, U$1.VIN@1, U$1.VIN@2
- net N$10: now also U$1.!CS, U$1.FB
- net N$2: now also U$1.DVDD
- net N$3: now also U$1.L1, U$1.VDD
- net N$4: now also U$1.ISENSOR, U$1.REFIN–
- net N$5: now also U$1.L2, U$1.REFIN+
- net N$6: now also U$1.D, U$1.RTDIN+; no longer C2.2, C3.2, U1.VDDCORE, U1.VDDCORE@1, U1.VDDOUT
- net N$7: now also U$1.G, U$1.RTDIN–, U$1.VAUX
- net N$8: now also U$1.FORCE–, U$1.S
Other:
- moved on the sheet: C2, C3

Commit message: Module updates
1. Fixed or added ports to the following modules: DC-DC Converter, RTD,
Ordnance, and Firing Chains
2. Fixed power pins within those modules
3. Minor updates to the DC-DC Converter regarding the connections to the
TPS63070
4. Moved the RTD's screw terminal block to the top level sheet
Parts:
- removed U$1: 2POS_SCREWTERM, CRAP Parts:2POS_SCREWTERM
- added J1: 2POS_SCREWTERM, CRAP Parts:2POS_SCREWTERM
- added J2: 4POS_SCREWTERM, CRAP Parts:4POS_SCREWTERM
Connections:
- removed net 3V3_OUT: U$1.VOUT@1, U$1.VOUT@2
- removed net N$11: U$1.EN, U$1.FORCE+, U$1.PS/SYNC
- removed net N$12: U$1.SCLK
- removed net N$13: U$1.SDI
- removed net N$14: U$1.!DRDY
- new net S+: C3.1
- new net S–: C3.2
- new net VCC: C1.1, C2.1
- net +3V3: now also C3.1, U1.VIN
- net GND: now also J1.P$2; no longer U$1.DGND, U$1.EP, U$1.FORCE2, U$1.GND, U$1.GND@1, U$1.GND@2, U$1.PGND
- net N$1: no longer U$1.BIAS, U$1.VIN@1, U$1.VIN@2
- net N$10: no longer U$1.!CS, U$1.FB
- net N$2: no longer C2.1, U$1.DVDD
- net N$3: no longer C1.1, C3.1, U$1.L1, U$1.VDD, U1.VIN
- net N$4: no longer U$1.ISENSOR, U$1.REFIN–
- net N$5: no longer U$1.L2, U$1.REFIN+
- net N$6: now also J2.P$1; no longer C3.1, U$1.D, U$1.RTDIN+
- net N$7: now also J2.P$2; no longer C3.2, U$1.G, U$1.RTDIN–, U$1.VAUX
- net N$8: now also J2.P$3; no longer U$1.FORCE–, U$1.S
- net N$9: now also J2.P$4; no longer U$1.P$2, U$1.PG, U$1.SDO
- net VCC_IN: now also J1.P$1; no longer U$1.P$1
Other:
- note added: "DESCRIPTION OF MODULE PINS ~CONT_EN: Enable pin to trigger continuity check operation CONT_STAT: Status of continuity check function. 1 indicates pyro connected ORD_PWR: Firing chain power (from capacitor bank) 3V3: Power to run digital I/O FIRE1: Upper NFET firing command FIRE2: Lower NFET firing command"
- note added: "FB2 is indeed going to GND"
- note added: "NOTE TO ROUTER: Put the following silkscreen text next to each pin: 1: EXC+ 2: S+ 3: S– 4: EXC–"
- note added: "NOTE TO THE ROUTER The configuration of the wires for EN and PS is how it should be routed. I.e., nothing should be between the final 0603 capacitor and the chip. See figure 8 of the datasheet."
- note added: "Question from Cooper: Is this SPI? I thought you added SPI...?"
- note added: "RBF power on/off"
- note added: "Reverse current protection"
- note added: "Still need to place a diode here"
- note added: "This is SPI and not I2C"
- note added: "VSEL can go straight to ground without a pulldown according to figure 8 of the datasheet."
- note removed: "FIRE1"
- note removed: "FIRE2"
- note removed: "J1"

Commit message: Modules, aesthetics, library fixes
1. Renamed Ordnance to Ordnance Power. Moved Firing chains from inside
this module to the top level schematic.
2. Added Breakwire module with pins. Nothing done inside the module
3. Added IMU module with pins. Nothing done inside the module
4. Increased soldermask expansion on TPS63070 per datasheet inside the
Texas.lbr
5. Fixed the header pin names, pin connections, reference designators,
and added a frame on the schematic
6. Got smaller diode array on Ordnance Power board per Evan's request
7. Moved Firing Circuits to top level schematic. Previously on Ordnance
Board
8. Grouped like items on the top level schematic and added a frame for
aesthetics and ease to finding components
Parts:
- added J3, J4, J5: 4POS_SCREWTERM, CRAP Parts:4POS_SCREWTERM
Connections:
- net ORD_PWR renamed N$99
- net GND: now also J1.P2; no longer J1.P$2
- net N$6: now also J2.P1; no longer J2.P$1
- net N$7: now also J2.P2; no longer J2.P$2
- net N$8: now also J2.P3; no longer J2.P$3
- net N$9: now also J2.P4; no longer J2.P$4
- net VCC_IN: now also J1.P1; no longer J1.P$1
Other:
- note added: "LED indicates caps are charged"
- note added: "NOTE TO ROUTER Put the following on the silkscreen next to each pin: 1: + 2: –"
- note added: "NOTE TO THE ROUTER Put "x+" and "x–" on the silkscreen, where x means the firing chain number."
- note added: "Need two 100 uF caps in parallel if only using one super capacitor"
- note added: "Ordnance Charging and Power Circuit Cooper Barry"
- note added: "POWER"
- note added: "PYRO"
- note added: "SENSORS"
- note added: "Top Level Schematic"
- note removed: "Ordnance Charging and Pyro Chain Connections Cooper Barry"
