File: GitHub Projects/CRAP Project/Flight Controller.sch (EAGLE design)
At the start: 10 parts, among them J1 2POS_SCREWTERM, J2 4POS_SCREWTERM, J3 4POS_SCREWTERM, J4 4POS_SCREWTERM, J5 4POS_SCREWTERM

Commit message: Added frames and MPU-9250 into IMU module
Also remade the board again because it broke.
Parts:
- removed J5: 4POS_SCREWTERM, CRAP Parts:4POS_SCREWTERM
Changed lines of the file:
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@@
 <?xml version="1.0" encoding="utf-8"?>
 <!DOCTYPE eagle SYSTEM "eagle.dtd">
-<eagle version="7.7.0">
+<eagle version="8.0.1">
 <drawing>
 <settings>
@@
 </variantdefs>
 <parts>
+<part name="FRAME1" library="frames" deviceset="A3L-LOC" device=""/>
 </parts>
 <sheets>
@@
 </plain>
 <instances>
+<instance part="FRAME1" gate="G$1" x="0" y="0"/>
 </instances>
 <busses>
@@
 </variantdefs>
 <parts>
+<part name="FRAME1" library="frames" deviceset="A3L-LOC" device=""/>
+<part name="U1" library="InvenSense" deviceset="MPU-9250" device=""/>
 </parts>
 <sheets>
@@
 </plain>
 <instances>
+<instance part="FRAME1" gate="G$1" x="0" y="0"/>
+<instance part="U1" gate="G$1" x="180.34" y="132.08"/>
 </instances>
 <busses>
@@
 <part name="GND14" library="supply1" deviceset="GND" device=""/>
 <part name="+3V14" library="supply1" deviceset="+3V3" device=""/>
-<part name="J5" library="CRAP Parts" deviceset="4POS_SCREWTERM" device=""/>
 </parts>
 <sheets>
@@
 <instance part="GND14" gate="1" x="-146.05" y="35.56"/>
 <instance part="+3V14" gate="G$1" x="-147.32" y="78.74"/>
-<instance part="J5" gate="G$1" x="-254" y="-129.54"/>
 </instances>
 <busses>

Commit message: Added Micron 1Gbit memory module
1. Changed all the text to the info layer
2. Added the Micron 1Gbit memory module
3. Routed power and ground to it
Connections:
- net +3V3: now also U1.VCC
Other:
- note added: "MS5611 Module Evan Swinney"
Changed lines of the file:
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@@
 <sheet>
 <plain>
+<text x="88.9" y="-114.3" size="1.778" layer="97">MS5611 Module
+Evan Swinney</text>
 </plain>
 <instances>
@@
 <sheet>
 <plain>
-<text x="-68.58" y="20.32" size="1.778" layer="91">The input and output capacitors
+<text x="-68.58" y="20.32" size="1.778" layer="97">The input and output capacitors
 are not of the same physical
 size! Place the 0603 nearest
 to the chip.</text>
-<text x="-104.14" y="-30.48" size="1.778" layer="91">RBF goes here connecting
+<text x="-104.14" y="-30.48" size="1.778" layer="97">RBF goes here connecting
 the MOSFET gate to ground
 via the resistor.</text>
-<text x="78.74" y="15.24" size="1.778" layer="91">Place the 10uF, 0603
+<text x="78.74" y="15.24" size="1.778" layer="97">Place the 10uF, 0603
 as close to the chip
 as possible</text>
-<text x="-200.66" y="10.16" size="1.778" layer="91">Header connections are not
+<text x="-200.66" y="10.16" size="1.778" layer="97">Header connections are not
 inside this module on purpose</text>
-<text x="10.16" y="-43.18" size="1.778" layer="91">FB2 is indeed going to GND</text>
-<text x="-66.04" y="-35.56" size="1.778" layer="91">NOTE TO THE ROUTER
+<text x="10.16" y="-43.18" size="1.778" layer="97">FB2 is indeed going to GND</text>
+<text x="-66.04" y="-35.56" size="1.778" layer="97">NOTE TO THE ROUTER
 The configuration of the wires
 for EN and PS is how it should
@@
 capacitor and the chip.
 See figure 8 of the datasheet.</text>
-<text x="-17.78" y="-33.02" size="1.778" layer="91">VSEL can go straight to ground
+<text x="-17.78" y="-33.02" size="1.778" layer="97">VSEL can go straight to ground
 without a pulldown according
 to figure 8 of the datasheet.</text>
-<text x="-152.4" y="25.4" size="1.778" layer="91">Reverse current protection</text>
-<text x="-109.22" y="22.86" size="1.778" layer="91">RBF power on/off</text>
+<text x="-152.4" y="25.4" size="1.778" layer="97">Reverse current protection</text>
+<text x="-109.22" y="22.86" size="1.778" layer="97">RBF power on/off</text>
 </plain>
 <instances>
@@
 </segment>
 </net>
+<net name="N$8" class="0">
+<segment>
+<wire x1="-40.64" y1="-15.24" x2="-33.02" y2="0" width="0.1524" layer="91"/>
+<wire x1="-33.02" y1="0" x2="-32.766" y2="-2.54" width="0.1524" layer="91"/>
+<wire x1="-33.02" y1="0" x2="-35.306" y2="-1.27" width="0.1524" layer="91"/>
+</segment>
+</net>
 </nets>
 </sheet>
@@
 <sheet>
 <plain>
-<text x="328.93" y="168.91" size="1.778" layer="91">Ordnance connections outside of
+<text x="328.93" y="168.91" size="1.778" layer="97">Ordnance connections outside of
 the firing chain, so we can use
 more than a 2-terminal block.</text>
-<text x="170.18" y="177.8" size="1.778" layer="91">Power in after diode array
+<text x="170.18" y="177.8" size="1.778" layer="97">Power in after diode array
 from super capacitors</text>
-<text x="147.32" y="201.93" size="1.778" layer="91">!CONT_EN
+<text x="147.32" y="201.93" size="1.778" layer="97">!CONT_EN
 Continuity Enable command</text>
-<text x="170.18" y="165.1" size="1.778" layer="91">CONT_STAT
+<text x="170.18" y="165.1" size="1.778" layer="97">CONT_STAT
 Continuity Status</text>
-<text x="33.02" y="63.5" size="1.778" layer="91">DESCRIPTION OF MODULE PINS
+<text x="33.02" y="63.5" size="1.778" layer="97">DESCRIPTION OF MODULE PINS
 ~CONT_EN: Enable pin to trigger continuity
      check operation
@@
 FIRE1: Upper NFET firing command
 FIRE2: Lower NFET firing command</text>
-<text x="217.17" y="191.77" size="1.778" layer="91">Still need to place a diode here</text>
+<text x="217.17" y="191.77" size="1.778" layer="97">Still need to place a diode here</text>
 </plain>
 <instances>
@@
 <sheet>
 <plain>
-<text x="-59.69" y="-1.27" size="1.778" layer="91">Sets current input
+<text x="-59.69" y="-1.27" size="1.778" layer="97">Sets current input
 limit to 0.3A</text>
-<text x="109.22" y="-93.98" size="1.778" layer="91">Ordnance Charging and Power Circuit
+<text x="109.22" y="-93.98" size="1.778" layer="97">Ordnance Charging and Power Circuit
 Cooper Barry</text>
 <text x="-34.29" y="57.15" size="1.778" layer="91">LTC3225</text>
-<text x="106.68" y="0" size="1.778" layer="91">LED indicates caps are charged</text>
-<text x="6.35" y="52.07" size="1.778" layer="91">Need two 100 uF caps
+<text x="106.68" y="0" size="1.778" layer="97">LED indicates caps are charged</text>
+<text x="6.35" y="52.07" size="1.778" layer="97">Need two 100 uF caps
 in parallel if only using
 one super capacitor</text>
@@
 <sheet>
 <plain>
-<text x="114.3" y="27.94" size="1.778" layer="91">Why 3 resistors in parallel? A 400R resistor
+<text x="114.3" y="27.94" size="1.778" layer="97">Why 3 resistors in parallel? A 400R resistor
 is not cheap, and 1.2k is a standard value
 in the E12 series. Also, the accuracy of the
@@
 of this set resistor, and 3 in parallel reduces
 the tolerance by 3x.</text>
-<text x="111.76" y="7.62" size="1.778" layer="91">NOTE TO THE ROUTER:
+<text x="111.76" y="7.62" size="1.778" layer="97">NOTE TO THE ROUTER:
 Wire these as Kelvin connections
 where the REFIN pins are the
 sensing terminals!</text>
-<text x="81.28" y="27.94" size="1.778" layer="91">The 10 M resistor is for fault
+<text x="81.28" y="27.94" size="1.778" layer="97">The 10 M resistor is for fault
 detection if one of the RTD
 wires breaks.</text>
-<text x="142.24" y="-25.4" size="1.778" layer="91">NOTE TO ROUTER:
+<text x="142.24" y="-25.4" size="1.778" layer="97">NOTE TO ROUTER:
 Put the following silkscreen
 text next to each pin:
@@
 2: S–
 1: EXC–</text>
-<text x="185.42" y="-111.76" size="1.778" layer="91">RTD Sensing Circuit
+<text x="185.42" y="-111.76" size="1.778" layer="97">RTD Sensing Circuit
 Cooper Barry</text>
 </plain>
@@
 <parts>
 <part name="FRAME1" library="frames" deviceset="A3L-LOC" device=""/>
+<part name="U1" library="micron" deviceset="MT29F1G01" device=""/>
+<part name="GND1" library="supply1" deviceset="GND" device=""/>
+<part name="GND2" library="supply1" deviceset="GND" device=""/>
+<part name="+3V1" library="supply1" deviceset="+3V3" device=""/>
+<part name="C1" library="rcl" deviceset="C-EU" device="C0603" value="0.1u"/>
 </parts>
 <sheets>
@@
 <instances>
 <instance part="FRAME1" gate="G$1" x="0" y="0"/>
+<instance part="U1" gate="G$1" x="190.5" y="127"/>
+<instance part="GND1" gate="1" x="215.9" y="111.76"/>
+<instance part="GND2" gate="1" x="134.62" y="119.38"/>
+<instance part="+3V1" gate="G$1" x="129.54" y="137.16"/>
+<instance part="C1" gate="G$1" x="134.62" y="129.54"/>
 </instances>
 <busses>
 </busses>
 <nets>
+<net name="GND" class="0">
+<segment>
+<pinref part="C1" gate="G$1" pin="2"/>
+<pinref part="GND2" gate="1" pin="GND"/>
+<wire x1="134.62" y1="121.92" x2="134.62" y2="124.46" width="0.1524" layer="91"/>
+</segment>
+<segment>
+<pinref part="U1" gate="G$1" pin="GND"/>
+<pinref part="GND1" gate="1" pin="GND"/>
+<wire x1="210.82" y1="121.92" x2="215.9" y2="121.92" width="0.1524" layer="91"/>
+<wire x1="215.9" y1="121.92" x2="215.9" y2="114.3" width="0.1524" layer="91"/>
+</segment>
+</net>
+<net name="+3V3" class="0">
+<segment>
+<pinref part="+3V1" gate="G$1" pin="+3V3"/>
+<pinref part="U1" gate="G$1" pin="VCC"/>
+<wire x1="129.54" y1="134.62" x2="134.62" y2="134.62" width="0.1524" layer="91"/>
+<pinref part="C1" gate="G$1" pin="1"/>
+<wire x1="134.62" y1="134.62" x2="170.18" y2="134.62" width="0.1524" layer="91"/>
+<wire x1="134.62" y1="132.08" x2="134.62" y2="134.62" width="0.1524" layer="91"/>
+<junction x="134.62" y="134.62"/>
+</segment>
+</net>
 </nets>
 </sheet>
@@
 <text x="166.37" y="-171.196" size="2.54" layer="94">Created by members of the CRAP team
 Space Hardware Club</text>
-<text x="-261.62" y="99.06" size="1.778" layer="91">NOTE TO ROUTER:
+<text x="-261.62" y="99.06" size="1.778" layer="97">NOTE TO ROUTER:
 Put the following silkscreen
 text next to each pin:
@@
 3: S–
 4: EXC–</text>
-<text x="-165.1" y="114.3" size="1.778" layer="91">This is SPI and not I2C</text>
-<text x="-125.73" y="13.97" size="1.778" layer="91" rot="MR0">Question from Cooper:
+<text x="-165.1" y="114.3" size="1.778" layer="97">This is SPI and not I2C</text>
+<text x="-125.73" y="13.97" size="1.778" layer="97" rot="MR0">Question from Cooper:
 Is this SPI? I thought
 you added SPI...?</text>
-<text x="-260.35" y="186.69" size="1.778" layer="91">NOTE TO ROUTER
+<text x="-260.35" y="186.69" size="1.778" layer="97">NOTE TO ROUTER
 Put the following on the
 silkscreen next to each pin:
@@
 <frame x1="152.4" y1="-43.18" x2="265.43" y2="220.98" columns="0" rows="0" layer="91" border-left="no" border-top="no" border-right="no" border-bottom="no"/>
 <text x="219.71" y="-38.1" size="6.4516" layer="91">PYRO</text>
-<text x="208.28" y="-179.07" size="3.556" layer="91">Top Level Schematic</text>
-<text x="228.6" y="87.63" size="1.778" layer="91">NOTE TO THE ROUTER
+<text x="208.28" y="-179.07" size="3.556" layer="97">Top Level Schematic</text>
+<text x="228.6" y="87.63" size="1.778" layer="97">NOTE TO THE ROUTER
 Put "x+" and "x–" on the
 silkscreen, where x means

Commit message: Added super cap part, did prelim board layout
1. Made a super capacitor part with a upright and folded variant.
2. Talked with Davis about the dimensions of the board and came to the
conclusion that 100mm tall will be alright.  Also speculated that 100mm
tall board would work with most club rockets, and confirmed with both
supersonic teams that 100mm tall would be able to fit.
3. Changed some of the modules in the upper level sheet to fit back on
the 0.1" grid, although some of the ports are still 0.05" off.
4. Renamed in the ordance sheet the long lines to PYRO+ and PYRO- to
allign with the module ports.
5. Attached PYRO+ and PYRO- in the top level sheet to the headers in the
same fashion each time
6. Named the nets of each firing circuit attachment to their
corresponding module and if they were + or -, e.g.: FC1+ or FC4-
7. On the silkscreen made + and - text on tPlace layer (top silkscreen
layer) and alligned with each firing pin.
Connections:
- removed net N$99: U1.COUT
- new net FC1+: J3.P1
- new net FC1-: J3.P2
- new net FC2+: J3.P3
- new net FC2-: J3.P4
- new net FC3+: J4.P1
- new net FC3-: J4.P2
- new net FC4+: J4.P3
- new net FC4-: J4.P4
- net GND: now also J1.P1
- net N$3: now also U1.COUT
- net N$6: now also J1.P2

Commit message: IMU, Breakwire, Firing Chain module updates
1. Added CES521 diode to diode.lbr
2. Added CES521 to breakwire and pyro firing chain modules
3. Basic wiring of IMU module

Issues needing to be resolved with Evan
1. Address of IMU. There is a dangling resistor ready for this on the
top level schematic.
2. What does FSYNC need to be wired to inside the IMU module?
3. The breakwire and firing chain modules have two pins that I want
connected internally but named separately. See comments inside these
modules for more information.
4. What value of resistors to use for the IMU I2C lines. Currently 2.2k
Parts:
- added J5: 4POS_SCREWTERM, CRAP Parts:4POS_SCREWTERM
- added R1: 10k, rcl:R-US_R0603
Connections:
- new net AD0: U1.AD0/SDO
- new net BW–: C1.1
- new net INT: U1.INT
- new net N$11: J5.P3
- new net N$12: J5.P4
- new net N$13: J5.P1
- new net PYRO+: R1.1
- new net PYRO–: C1.1
- new net SCL: U1.SCL/SCLK
- new net SDA: U1.SDA/SDI
- net +3V3: now also R1.2, U1.REGOUT, U1.RESV
- net GND: now also U1.RESV/GND
- net N$1: now also R1.1, R1.2
- net N$10: now also J5.P2
- net N$2: now also R1.2
- net N$3: now also R1.2
- net N$4: now also R1.1
- net N$5: now also R1.1
- net VCC: now also C3.1, R1.2, U1.CS, U1.VDD
Other:
- note added: "ISSUE: I want to have two separate ports on the module for (CONT_STAT & PYRO–) and (ORD_PWR & PRYO+), but I cannot have two names for a net. How should this be worked around? I don't want to use a 0 Ohm resistor. Make a small via that connects two nets?"
- note added: "ISSUE: I want two pins on the module named BW– and BW_STAT, but I cannot have two names for the same net."
- note added: "NOTE TO ROUTER: Place the following text next to each pin 1. 1+ 2. 1– 3. 2+ 4. 2–"
- note added: "What do you want FSYNC (11) connected to?"
- note removed: "Still need to place a diode here"
- moved on the sheet: J1

Commit message: Added H3LIS100DL
Added the H3LIS100DL to the ST-microelectronics library along with a
3x3mm TFLGA-16 package. This device is in the HIGH_G module under
Sensors. Things for Evan to consider on this push:
1. Frame needed for the HIGH_G module schematic
2. Data communication for H3LIS100DL: SPI or I2C?
2a. If I2C, which address? Currently a resistor on the top level
schematic pulling it to 0.
3. Please check my footprint. Once again, I have more evidence for my
hate of ST: they did not provide a recommended solder footprint for the
TFLGA package. Therefore, I took the mechanical pad side of 0.35x0.25
and added 0.1 mm to each dimension to yield 0.45x0.35 (according to
their note TN0018) . I am fairly certain I centered the pads on the
pins. Yes, that is a purposeful solder mask expansion.
Parts:
- added R2: 10k, rcl:R-US_R0603
Connections:
- new net FIRE2: R2.2
- new net INT1: U1.INT1
- new net INT2: U1.INT2
- new net N$14: R1.2
- new net N$15: R2.2
- new net SA0/SDO: U1.SA0/SDO
- new net SCL/SPC: U1.SCL/SPC
- new net SDA/SDI: U1.SDA/SDI
- net CS: now also U1.CS
- net GND: now also R1.1, R2.1, U1.GND@3, U1.GND@4, U1.RES@2
- net N$1: now also R2.2
- net N$4: now also R2.1
- net N$6: now also R2.2
- net N$8: now also R2.1
- net SCL: now also R2.1
- net VCC: now also R2.2, U1.RES@1, U1.VDD_IO
Other:
- note added: "CS needs to be 0: SPI enables 1: I2C bus"
- note added: "INT pins can be push-pull"
- note added: "Place C2 nearest pin 1 and C3 nearest pin 14 (or swap, I don't care). As long as the 0603, 0.1 uF caps are closest to the pin on the device."
- moved on the sheet: R1
