File: GitHub Projects/CRAP Project/Flight Controller.sch (EAGLE design)
At the start: 12 parts, among them J1 2POS_SCREWTERM, J2 4POS_SCREWTERM, J3 4POS_SCREWTERM, J4 4POS_SCREWTERM, J5 4POS_SCREWTERM

Commit message: Ordnance power updates
1. Fixed PGOOD LED on Ordnance Power module
2. Wired output capacitors on Ordnance Power. This is a single super-cap
configuration where two 100uF caps in series are needed fro the
balancing circuitry.
3. Added a frame to the HIGH_G module

Another issue discovered:
1. Need USB connection. There are no micro USBs in the library (unless
I'm blind?)
Connections:
- net +3V3: now also R2.2
- net N$10: no longer U1.CX
- net N$4: now also U1.PGOOD
- net N$7: now also U1.CX
- net N$8: no longer R2.1, U1.PGOOD
Other:
- note added: "Open drain output"
Changed lines of the file:
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@@
 <setting verticaltext="up"/>
 </settings>
-<grid distance="0.05" unitdist="inch" unit="inch" style="lines" multiple="1" display="no" altdistance="0.01" altunitdist="inch" altunit="inch"/>
+<grid distance="0.1" unitdist="inch" unit="inch" style="lines" multiple="1" display="no" altdistance="0.01" altunitdist="inch" altunit="inch"/>
 <layers>
 <layer number="1" name="Top" color="4" fill="1" visible="no" active="no"/>
@@
 <part name="C3" library="rcl" deviceset="C-EU" device="C0603" value="1u"/>
 <part name="R1" library="resistor" deviceset="R-US_" device="R0603" value="10k"/>
-<part name="R2" library="resistor" deviceset="R-US_" device="R0603" value="100k"/>
+<part name="R2" library="resistor" deviceset="R-US_" device="R0603" value="2.2k"/>
 <part name="R3" library="resistor" deviceset="R-US_" device="R0603" value="12k"/>
-<part name="R4" library="resistor" deviceset="R-US_" device="R0603" value="10k"/>
-<part name="C4" library="rcl" deviceset="C-EU" device="C0603" value="1u"/>
+<part name="C4" library="rcl" deviceset="C-EU" device="C0603" value="0.1u"/>
 <part name="FRAME1" library="frames" deviceset="A3L-LOC" device=""/>
 <part name="GND1" library="supply1" deviceset="GND" device=""/>
@@
 <part name="C5" library="CRAP Parts" deviceset="AVX_1F_5V" device="FOLDED"/>
 <part name="GND5" library="supply1" deviceset="GND" device=""/>
+<part name="+3V2" library="supply1" deviceset="+3V3" device=""/>
+<part name="D2" library="led" deviceset="LED" device="CHIP-LED0603" value="LTST-C193KRKT-2A"/>
+<part name="GND6" library="supply1" deviceset="GND" device=""/>
+<part name="C6" library="rcl" deviceset="C-EU" device="C1206" value="100u"/>
+<part name="C7" library="rcl" deviceset="C-EU" device="C1206" value="100u"/>
+<part name="GND7" library="supply1" deviceset="GND" device=""/>
 </parts>
 <sheets>
@@
 Cooper Barry</text>
 <text x="-33.02" y="55.88" size="1.778" layer="91">LTC3225</text>
-<text x="106.68" y="0" size="1.778" layer="97">LED indicates caps are charged</text>
+<text x="111.76" y="-20.32" size="1.778" layer="97">LED indicates caps are charged</text>
 <text x="7.62" y="50.8" size="1.778" layer="97">Need two 100 uF caps
 in parallel if only using
 one super capacitor</text>
+<text x="0" y="0" size="1.778" layer="97">Open drain output</text>
 </plain>
 <instances>
@@
 <attribute name="VALUE" x="-69.85" y="33.782" size="1.778" layer="96" rot="R180"/>
 </instance>
-<instance part="R2" gate="G$1" x="86.36" y="30.48" smashed="yes" rot="R90">
-<attribute name="NAME" x="85.09" y="34.0614" size="1.778" layer="95" rot="R180"/>
-<attribute name="VALUE" x="85.09" y="31.242" size="1.778" layer="96" rot="R180"/>
+<instance part="R2" gate="G$1" x="91.44" y="10.16" smashed="yes" rot="R90">
+<attribute name="NAME" x="90.17" y="13.7414" size="1.778" layer="95" rot="R180"/>
+<attribute name="VALUE" x="90.17" y="10.922" size="1.778" layer="96" rot="R180"/>
 </instance>
 <instance part="R3" gate="G$1" x="-33.02" y="0" smashed="yes" rot="R90">
@@
 <attribute name="VALUE" x="-34.29" y="0.762" size="1.778" layer="96" rot="R180"/>
 </instance>
-<instance part="R4" gate="G$1" x="99.06" y="22.86" smashed="yes" rot="R180">
-<attribute name="NAME" x="95.25" y="24.3586" size="1.778" layer="95"/>
-<attribute name="VALUE" x="95.25" y="19.558" size="1.778" layer="96"/>
-</instance>
-<instance part="C4" gate="G$1" x="86.36" y="17.78"/>
+<instance part="C4" gate="G$1" x="91.44" y="-2.54"/>
 <instance part="FRAME1" gate="G$1" x="-180.34" y="-111.76"/>
 <instance part="GND1" gate="1" x="-33.02" y="-10.16"/>
 <instance part="GND2" gate="1" x="-91.44" y="22.86"/>
-<instance part="GND3" gate="1" x="86.36" y="7.62"/>
+<instance part="GND3" gate="1" x="91.44" y="-15.24"/>
 <instance part="GND4" gate="1" x="-15.24" y="13.97"/>
 <instance part="+3V1" gate="G$1" x="-91.44" y="50.8"/>
 <instance part="D1" gate="G$1" x="48.26" y="40.64"/>
-<instance part="C5" gate="G$1" x="33.02" y="38.1"/>
-<instance part="GND5" gate="1" x="33.02" y="27.94"/>
+<instance part="C5" gate="G$1" x="33.02" y="30.48"/>
+<instance part="GND5" gate="1" x="33.02" y="10.16"/>
+<instance part="+3V2" gate="G$1" x="91.44" y="22.86"/>
+<instance part="D2" gate="G$1" x="116.84" y="-2.54"/>
+<instance part="GND6" gate="1" x="116.84" y="-15.24"/>
+<instance part="C6" gate="G$1" x="20.32" y="35.56"/>
+<instance part="C7" gate="G$1" x="20.32" y="22.86"/>
+<instance part="GND7" gate="1" x="20.32" y="10.16"/>
 </instances>
 <busses>
@@
 <pinref part="R3" gate="G$1" pin="2"/>
 <wire x1="-33.02" y1="7.62" x2="-33.02" y2="5.08" width="0.1524" layer="91"/>
-</segment>
-</net>
-<net name="N$10" class="0">
-<segment>
-<pinref part="U1" gate="G$1" pin="CX"/>
-<wire x1="-17.78" y1="38.1" x2="17.78" y2="38.1" width="0.1524" layer="91"/>
-</segment>
-</net>
-<net name="N$8" class="0">
-<segment>
-<pinref part="R4" gate="G$1" pin="2"/>
-<pinref part="U1" gate="G$1" pin="PGOOD"/>
-<wire x1="93.98" y1="22.86" x2="86.36" y2="22.86" width="0.1524" layer="91"/>
-<pinref part="R2" gate="G$1" pin="1"/>
-<pinref part="C4" gate="G$1" pin="1"/>
-<wire x1="86.36" y1="22.86" x2="-17.78" y2="22.86" width="0.1524" layer="91"/>
-<wire x1="86.36" y1="25.4" x2="86.36" y2="22.86" width="0.1524" layer="91"/>
-<junction x="86.36" y="22.86"/>
-<wire x1="86.36" y1="22.86" x2="86.36" y2="20.32" width="0.1524" layer="91"/>
 </segment>
 </net>
@@
 <pinref part="GND3" gate="1" pin="GND"/>
 <pinref part="C4" gate="G$1" pin="2"/>
-<wire x1="86.36" y1="10.16" x2="86.36" y2="12.7" width="0.1524" layer="91"/>
+<wire x1="91.44" y1="-12.7" x2="91.44" y2="-7.62" width="0.1524" layer="91"/>
 </segment>
 <segment>
@@
 <pinref part="C5" gate="G$1" pin="-"/>
 <pinref part="GND5" gate="1" pin="GND"/>
-<wire x1="33.02" y1="33.02" x2="33.02" y2="30.48" width="0.1524" layer="91"/>
+<wire x1="33.02" y1="25.4" x2="33.02" y2="12.7" width="0.1524" layer="91"/>
+</segment>
+<segment>
+<pinref part="D2" gate="G$1" pin="C"/>
+<wire x1="116.84" y1="-7.62" x2="116.84" y2="-12.7" width="0.1524" layer="91"/>
+<pinref part="GND6" gate="1" pin="GND"/>
+</segment>
+<segment>
+<pinref part="C7" gate="G$1" pin="2"/>
+<pinref part="GND7" gate="1" pin="GND"/>
+<wire x1="20.32" y1="17.78" x2="20.32" y2="12.7" width="0.1524" layer="91"/>
 </segment>
 </net>
@@
 <junction x="-91.44" y="43.18"/>
 </segment>
+<segment>
+<pinref part="R2" gate="G$1" pin="2"/>
+<pinref part="+3V2" gate="G$1" pin="+3V3"/>
+<wire x1="91.44" y1="15.24" x2="91.44" y2="20.32" width="0.1524" layer="91"/>
+</segment>
 </net>
 <net name="N$3" class="0">
@@
 <wire x1="43.18" y1="38.1" x2="46.99" y2="38.1" width="0.1524" layer="91"/>
 <pinref part="U1" gate="G$1" pin="COUT"/>
-<wire x1="-17.78" y1="43.18" x2="33.02" y2="43.18" width="0.1524" layer="91"/>
+<wire x1="-17.78" y1="43.18" x2="20.32" y2="43.18" width="0.1524" layer="91"/>
 <junction x="43.18" y="43.18"/>
 <pinref part="C5" gate="G$1" pin="+"/>
+<wire x1="20.32" y1="43.18" x2="33.02" y2="43.18" width="0.1524" layer="91"/>
 <wire x1="33.02" y1="43.18" x2="43.18" y2="43.18" width="0.1524" layer="91"/>
-<wire x1="33.02" y1="40.64" x2="33.02" y2="43.18" width="0.1524" layer="91"/>
+<wire x1="33.02" y1="33.02" x2="33.02" y2="43.18" width="0.1524" layer="91"/>
 <junction x="33.02" y="43.18"/>
+<pinref part="C6" gate="G$1" pin="1"/>
+<wire x1="20.32" y1="38.1" x2="20.32" y2="43.18" width="0.1524" layer="91"/>
+<junction x="20.32" y="43.18"/>
+</segment>
+</net>
+<net name="N$4" class="0">
+<segment>
+<pinref part="D2" gate="G$1" pin="A"/>
+<wire x1="116.84" y1="2.54" x2="116.84" y2="0" width="0.1524" layer="91"/>
+<pinref part="R2" gate="G$1" pin="1"/>
+<pinref part="C4" gate="G$1" pin="1"/>
+<wire x1="91.44" y1="5.08" x2="91.44" y2="2.54" width="0.1524" layer="91"/>
+<junction x="91.44" y="2.54"/>
+<wire x1="91.44" y1="2.54" x2="91.44" y2="0" width="0.1524" layer="91"/>
+<wire x1="91.44" y1="2.54" x2="-2.54" y2="2.54" width="0.1524" layer="91"/>
+<wire x1="-2.54" y1="2.54" x2="-2.54" y2="22.86" width="0.1524" layer="91"/>
+<pinref part="U1" gate="G$1" pin="PGOOD"/>
+<wire x1="-2.54" y1="22.86" x2="-17.78" y2="22.86" width="0.1524" layer="91"/>
+<wire x1="116.84" y1="2.54" x2="91.44" y2="2.54" width="0.1524" layer="91"/>
+</segment>
+</net>
+<net name="N$7" class="0">
+<segment>
+<pinref part="C6" gate="G$1" pin="2"/>
+<pinref part="C7" gate="G$1" pin="1"/>
+<wire x1="20.32" y1="30.48" x2="20.32" y2="27.94" width="0.1524" layer="91"/>
+<wire x1="20.32" y1="27.94" x2="20.32" y2="25.4" width="0.1524" layer="91"/>
+<wire x1="20.32" y1="27.94" x2="0" y2="27.94" width="0.1524" layer="91"/>
+<wire x1="0" y1="27.94" x2="0" y2="38.1" width="0.1524" layer="91"/>
+<pinref part="U1" gate="G$1" pin="CX"/>
+<wire x1="0" y1="38.1" x2="-17.78" y2="38.1" width="0.1524" layer="91"/>
+<junction x="20.32" y="27.94"/>
 </segment>
 </net>
@@
 <part name="C3" library="rcl" deviceset="C-EU" device="C0603" value="0.1u"/>
 <part name="GND2" library="supply1" deviceset="GND" device=""/>
+<part name="FRAME1" library="frames" deviceset="A3L-LOC" device=""/>
 </parts>
 <sheets>
@@
 <instance part="C3" gate="G$1" x="27.94" y="36.83"/>
 <instance part="GND2" gate="1" x="10.16" y="24.13"/>
+<instance part="FRAME1" gate="G$1" x="-157.48" y="-114.3"/>
 </instances>
 <busses>

Commit message: Ordnance & Breakwire modules fixes
1. In the Ordnance module: combined the PYRO+ and PWR to the same pin
and called PWR/PYRO+. This is the ordnance power from the super caps.
2. In the Ordnance module: combined CONT_STAT and PYRO– to the same pin
and called CONT_STAT/PYRO–. Outside the modules on the top level
schematic, I added long wires from this pin going to the left of each
module. This is also the digital line for sensing continuity status of
the ordnance lines.
3. In the Breakwire module, combined BW_STAT and BW– to the same pin and
called BW_STAT/BW–. Outside the module on the top level schematic, I
made long lines from this pin to the right of each module. This is the
digital input for sensing the breakwire status (open or closed).
Connections:
- net FC2- renamed FC1-1
- net FC4- renamed FC1-3
- net PYRO+ renamed PWR/PYRO+
- removed net BW–: C1.1
- removed net FC1+: J3.P1
- removed net FC3+: J4.P1
- removed net PYRO–: C1.1
- new net +12V: J3.P1, J4.P1
- new net BW_STAT/BW–: C1.1
- new net CONT_STAT/PYRO–: C1.1
Other:
- note added: "Place the USB here. Positive goes to PWR_IN and negative to GND. Note, this does not use diode steering, so the battery cannot be connected when powering through the USB. I don't care what you do with the data lines."
- note removed: "ISSUE: I want to have two separate ports on the module for (CONT_STAT & PYRO–) and (ORD_PWR & PRYO+), but I cannot have two names for a net. How should this be worked around? I don't want to use a 0 Ohm resistor. Make a small via that connects two nets?"
- note removed: "Question from Cooper: Is this SPI? I thought you added SPI...?"

Commit message: Major changes
1. Cleaned up master level sheet
2. Changed MS5611 from SPI to I2C
3. Routed a lot
4. Changed MPU9250 power structure on top level (was broken)
5. Added serial communication lines to microcontroller
Connections:
- removed net MISO: U1.SDO
- removed net MOSI: U1.SDI/SDA
- removed net SCLK: U1.SCLK
- new net GPS_RX: U1.PA13
- new net GPS_TX: U1.PA12
- new net MPU9250_SCL: U1.PA9
- new net MPU9250_SDA: U1.PA10
- new net MS5611_SCL: U1.PB2
- new net MS5611_SDA: U1.PB3
- new net N$20: U1.PA5
- new net N$21: U1.PA6
- new net SCL/SCLK: R2.1, U1.SCLK
- new net VIN: C1.1, C2.1, C3.1
- new net XBEE_RX: U1.PA28
- new net XBEE_TX: U1.PA27
- net +3V3: now also U1.CS, U1.PS
- net CS: no longer U1.CSB@1, U1.CSB@2
- net GND: now also U1.CSB@1, U1.CSB@2; no longer U1.PS
- net N$1: no longer C1.1, C3.1
- net SDA: now also R1.1, U1.SDI/SDA
- net VCC: no longer R2.2, U1.CS
Other:
- note added: "BW1_Status"
- note added: "BW2_Status"
- note added: "CSB = 0 On MS5611, Address is !Address, so the real address is actually 0bxxxxxxx1."
- note added: "NOTE TO ROUTER: Place the following text next to each pin 1. B1+ 2. B1– 3. B2+ 4. B2–"
- note added: "USART5 Module"
- note added: "USART7 Module"
- note removed: "MS5611 Module Evan Swinney"
- note removed: "NOTE TO ROUTER: Place the following text next to each pin 1. 1+ 2. 1– 3. 2+ 4. 2–"
- moved on the sheet: J5, JP1, R1, R2
