File: GitHub Projects/CRAP Project/Flight Controller.sch (EAGLE design)
At the start: 24 parts, among them J1 2POS_SCREWTERM, J2 4POS_SCREWTERM, J3 4POS_SCREWTERM, J4 4POS_SCREWTERM, J5 4POS_SCREWTERM

Commit message: Minor Changes to some routing
Having problems with using the alternate grid.  Routing engine will not
allow me to route on the alternate grid, which has stopped progress for
the time being.
Parts:
- U1: value (none) -> G55J19
Connections:
- net +3V3: now also U1.RES@1, U1.VDD_IO
- net VCC: no longer C3.1, R1.2, U1.RES@1, U1.VDD, U1.VDD_IO
Changed lines of the file:
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@@
 <?xml version="1.0" encoding="utf-8"?>
 <!DOCTYPE eagle SYSTEM "eagle.dtd">
-<eagle version="8.1.0">
+<eagle version="8.2.2">
 <drawing>
 <settings>
@@
 <grid distance="0.1" unitdist="inch" unit="inch" style="lines" multiple="1" display="no" altdistance="0.01" altunitdist="inch" altunit="inch"/>
 <layers>
-<layer number="1" name="Top" color="4" fill="1" visible="no" active="no"/>
-<layer number="2" name="Route2" color="1" fill="3" visible="no" active="no"/>
-<layer number="3" name="Route3" color="4" fill="3" visible="no" active="no"/>
-<layer number="4" name="Route4" color="1" fill="4" visible="no" active="no"/>
-<layer number="5" name="Route5" color="4" fill="4" visible="no" active="no"/>
-<layer number="6" name="Route6" color="1" fill="8" visible="no" active="no"/>
-<layer number="7" name="Route7" color="4" fill="8" visible="no" active="no"/>
-<layer number="8" name="Route8" color="1" fill="2" visible="no" active="no"/>
-<layer number="9" name="Route9" color="4" fill="2" visible="no" active="no"/>
-<layer number="10" name="Route10" color="1" fill="7" visible="no" active="no"/>
-<layer number="11" name="Route11" color="4" fill="7" visible="no" active="no"/>
-<layer number="12" name="Route12" color="1" fill="5" visible="no" active="no"/>
-<layer number="13" name="Route13" color="4" fill="5" visible="no" active="no"/>
-<layer number="14" name="Route14" color="1" fill="6" visible="no" active="no"/>
-<layer number="15" name="Route15" color="4" fill="6" visible="no" active="no"/>
-<layer number="16" name="Bottom" color="1" fill="1" visible="no" active="no"/>
-<layer number="17" name="Pads" color="2" fill="1" visible="no" active="no"/>
-<layer number="18" name="Vias" color="2" fill="1" visible="no" active="no"/>
-<layer number="19" name="Unrouted" color="6" fill="1" visible="no" active="no"/>
-<layer number="20" name="Dimension" color="15" fill="1" visible="no" active="no"/>
-<layer number="21" name="tPlace" color="7" fill="1" visible="no" active="no"/>
-<layer number="22" name="bPlace" color="7" fill="1" visible="no" active="no"/>
-<layer number="23" name="tOrigins" color="15" fill="1" visible="no" active="no"/>
-<layer number="24" name="bOrigins" color="15" fill="1" visible="no" active="no"/>
-<layer number="25" name="tNames" color="7" fill="1" visible="no" active="no"/>
-<layer number="26" name="bNames" color="7" fill="1" visible="no" active="no"/>
-<layer number="27" name="tValues" color="7" fill="1" visible="no" active="no"/>
-<layer number="28" name="bValues" color="7" fill="1" visible="no" active="no"/>
+<layer number="1" name="Top" color="4" fill="1" visible="yes" active="no"/>
+<layer number="2" name="Route2" color="1" fill="3" visible="yes" active="no"/>
+<layer number="3" name="Route3" color="4" fill="3" visible="yes" active="no"/>
+<layer number="4" name="Route4" color="1" fill="4" visible="yes" active="no"/>
+<layer number="5" name="Route5" color="4" fill="4" visible="yes" active="no"/>
+<layer number="6" name="Route6" color="1" fill="8" visible="yes" active="no"/>
+<layer number="7" name="Route7" color="4" fill="8" visible="yes" active="no"/>
+<layer number="8" name="Route8" color="1" fill="2" visible="yes" active="no"/>
+<layer number="9" name="Route9" color="4" fill="2" visible="yes" active="no"/>
+<layer number="10" name="Route10" color="1" fill="7" visible="yes" active="no"/>
+<layer number="11" name="Route11" color="4" fill="7" visible="yes" active="no"/>
+<layer number="12" name="Route12" color="1" fill="5" visible="yes" active="no"/>
+<layer number="13" name="Route13" color="4" fill="5" visible="yes" active="no"/>
+<layer number="14" name="Route14" color="1" fill="6" visible="yes" active="no"/>
+<layer number="15" name="Route15" color="4" fill="6" visible="yes" active="no"/>
+<layer number="16" name="Bottom" color="1" fill="1" visible="yes" active="no"/>
+<layer number="17" name="Pads" color="2" fill="1" visible="yes" active="no"/>
+<layer number="18" name="Vias" color="2" fill="1" visible="yes" active="no"/>
+<layer number="19" name="Unrouted" color="6" fill="1" visible="yes" active="no"/>
+<layer number="20" name="Dimension" color="15" fill="1" visible="yes" active="no"/>
+<layer number="21" name="tPlace" color="7" fill="1" visible="yes" active="no"/>
+<layer number="22" name="bPlace" color="7" fill="1" visible="yes" active="no"/>
+<layer number="23" name="tOrigins" color="15" fill="1" visible="yes" active="no"/>
+<layer number="24" name="bOrigins" color="15" fill="1" visible="yes" active="no"/>
+<layer number="25" name="tNames" color="7" fill="1" visible="yes" active="no"/>
+<layer number="26" name="bNames" color="7" fill="1" visible="yes" active="no"/>
+<layer number="27" name="tValues" color="7" fill="1" visible="yes" active="no"/>
+<layer number="28" name="bValues" color="7" fill="1" visible="yes" active="no"/>
 <layer number="29" name="tStop" color="7" fill="3" visible="no" active="no"/>
 <layer number="30" name="bStop" color="7" fill="6" visible="no" active="no"/>
@@
 <layer number="35" name="tGlue" color="7" fill="4" visible="no" active="no"/>
 <layer number="36" name="bGlue" color="7" fill="5" visible="no" active="no"/>
-<layer number="37" name="tTest" color="7" fill="1" visible="no" active="no"/>
-<layer number="38" name="bTest" color="7" fill="1" visible="no" active="no"/>
+<layer number="37" name="tTest" color="7" fill="1" visible="yes" active="no"/>
+<layer number="38" name="bTest" color="7" fill="1" visible="yes" active="no"/>
 <layer number="39" name="tKeepout" color="4" fill="11" visible="no" active="no"/>
 <layer number="40" name="bKeepout" color="1" fill="11" visible="no" active="no"/>
@@
 <layer number="44" name="Drills" color="7" fill="1" visible="no" active="no"/>
 <layer number="45" name="Holes" color="7" fill="1" visible="no" active="no"/>
-<layer number="46" name="Milling" color="3" fill="1" visible="no" active="no"/>
-<layer number="47" name="Measures" color="7" fill="1" visible="no" active="no"/>
-<layer number="48" name="Document" color="7" fill="1" visible="no" active="no"/>
-<layer number="49" name="Reference" color="7" fill="1" visible="no" active="no"/>
-<layer number="51" name="tDocu" color="7" fill="1" visible="no" active="no"/>
-<layer number="52" name="bDocu" color="7" fill="1" visible="no" active="no"/>
+<layer number="46" name="Milling" color="3" fill="1" visible="yes" active="no"/>
+<layer number="47" name="Measures" color="7" fill="1" visible="yes" active="no"/>
+<layer number="48" name="Document" color="7" fill="1" visible="yes" active="no"/>
+<layer number="49" name="Reference" color="7" fill="1" visible="yes" active="no"/>
+<layer number="51" name="tDocu" color="7" fill="1" visible="yes" active="no"/>
+<layer number="52" name="bDocu" color="7" fill="1" visible="yes" active="no"/>
 <layer number="90" name="Modules" color="5" fill="1" visible="yes" active="yes"/>
 <layer number="91" name="Nets" color="2" fill="1" visible="yes" active="yes"/>
@@
 </variantdefs>
 <parts>
-<part name="U1" library="linear-technology" deviceset="LTC3225" device=""/>
+<part name="U1" library="linear-technology" deviceset="LTC3225" device="" value="LTC3225"/>
 <part name="C1" library="rcl" deviceset="C-EU" device="C0805" value="2.2u"/>
 <part name="C2" library="rcl" deviceset="C-EU" device="C0402" value="1u"/>
@@
 </busses>
 <nets>
-<net name="VCC" class="0">
+<net name="+3V3" class="0">
 <segment>
 <pinref part="R1" gate="G$1" pin="2"/>
 <pinref part="+3V1" gate="G$1" pin="+3V3"/>
 <wire x1="177.8" y1="139.7" x2="177.8" y2="144.78" width="0.1524" layer="91"/>
-<label x="177.8" y="142.24" size="1.778" layer="95"/>
 </segment>
 </net>
@@
 <parts>
 <part name="FRAME1" library="frames" deviceset="A3L-LOC" device=""/>
-<part name="U1" library="InvenSense" deviceset="MPU-9250" device=""/>
+<part name="U1" library="InvenSense" deviceset="MPU-9250" device="" value="MPU9250"/>
 <part name="GND1" library="supply1" deviceset="GND" device=""/>
 <part name="C1" library="rcl" deviceset="C-EU" device="C0603" value="0.1u"/>
@@
 </segment>
 </net>
-<net name="VCC" class="0">
+<net name="+3V3" class="0">
 <segment>
 <pinref part="+3V1" gate="G$1" pin="+3V3"/>
@@
 </variantdefs>
 <parts>
-<part name="U1" library="Measurement Specialties" deviceset="MS5611" device=""/>
+<part name="U1" library="Measurement Specialties" deviceset="MS5611" device="" value="MS5611"/>
 <part name="C1" library="resistor" deviceset="C-EU" device="C0603" value="100n"/>
 <part name="GND1" library="supply1" deviceset="GND" device=""/>
@@
 </modules>
 <parts>
-<part name="U1" library="atmel" deviceset="ATSAMG55J19" device=""/>
+<part name="U1" library="atmel" deviceset="ATSAMG55J19" device="" value="G55J19"/>
 <part name="JP1" library="atmel" deviceset="AVR_JTAG" device=""/>
 <part name="GND1" library="supply1" deviceset="GND" device=""/>

Commit message: Major revisions
1. Made board 30mm taller to allow for more space in cramped enviroment.
Deemed absolutely critical.
2. Majorly changed the power turn-on and turn-off MOSFETs design and
location to clear up room in the mid-board area
3. Moved the super capacitor nearer to the top of the extended section,
and also made it have a verticle orientation; should allow for better
handling of vertical Gs
4. Moved the super-capacitor charging circuitry in the extra space under
the super-cap.  Fits nicely in a small area now.
5. Created Vishay.lbr, Adafruit.lbr, nkk.lbr, and semtech.lbr
6. Added common SMT pads to Semtech.lbr and Vishay.lbr
7. Created MOSFETs in Vishay.lbr
8.Created MOSFETs in semtech.lbr
9. Completely routed the GPS and passives; just needs UART connections
to the uC now
10. Changed the DRC (Design Rules) to better reflect the capabilities of
Advanced Circuit's $33/board abilities.  Changes are mostly downsizing
the rules to 7mil of smallest hole, trace, and spacing between copper to
copper
11. Modified all vias in tight locations and low power consumption roles
to be a 7mil (0.18mm, rounded) drill hole
Connections:
- net N$2: no longer R1.2
Changed lines of the file:
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@@
 <grid distance="0.1" unitdist="inch" unit="inch" style="lines" multiple="1" display="no" altdistance="0.01" altunitdist="inch" altunit="inch"/>
 <layers>
-<layer number="1" name="Top" color="4" fill="1" visible="yes" active="no"/>
-<layer number="2" name="Route2" color="1" fill="3" visible="yes" active="no"/>
-<layer number="3" name="Route3" color="4" fill="3" visible="yes" active="no"/>
-<layer number="4" name="Route4" color="1" fill="4" visible="yes" active="no"/>
-<layer number="5" name="Route5" color="4" fill="4" visible="yes" active="no"/>
-<layer number="6" name="Route6" color="1" fill="8" visible="yes" active="no"/>
-<layer number="7" name="Route7" color="4" fill="8" visible="yes" active="no"/>
-<layer number="8" name="Route8" color="1" fill="2" visible="yes" active="no"/>
-<layer number="9" name="Route9" color="4" fill="2" visible="yes" active="no"/>
-<layer number="10" name="Route10" color="1" fill="7" visible="yes" active="no"/>
-<layer number="11" name="Route11" color="4" fill="7" visible="yes" active="no"/>
-<layer number="12" name="Route12" color="1" fill="5" visible="yes" active="no"/>
-<layer number="13" name="Route13" color="4" fill="5" visible="yes" active="no"/>
-<layer number="14" name="Route14" color="1" fill="6" visible="yes" active="no"/>
-<layer number="15" name="Route15" color="4" fill="6" visible="yes" active="no"/>
-<layer number="16" name="Bottom" color="1" fill="1" visible="yes" active="no"/>
-<layer number="17" name="Pads" color="2" fill="1" visible="yes" active="no"/>
-<layer number="18" name="Vias" color="2" fill="1" visible="yes" active="no"/>
-<layer number="19" name="Unrouted" color="6" fill="1" visible="yes" active="no"/>
-<layer number="20" name="Dimension" color="15" fill="1" visible="yes" active="no"/>
-<layer number="21" name="tPlace" color="7" fill="1" visible="yes" active="no"/>
-<layer number="22" name="bPlace" color="7" fill="1" visible="yes" active="no"/>
-<layer number="23" name="tOrigins" color="15" fill="1" visible="yes" active="no"/>
-<layer number="24" name="bOrigins" color="15" fill="1" visible="yes" active="no"/>
-<layer number="25" name="tNames" color="7" fill="1" visible="yes" active="no"/>
-<layer number="26" name="bNames" color="7" fill="1" visible="yes" active="no"/>
-<layer number="27" name="tValues" color="7" fill="1" visible="yes" active="no"/>
-<layer number="28" name="bValues" color="7" fill="1" visible="yes" active="no"/>
+<layer number="1" name="Top" color="4" fill="1" visible="no" active="no"/>
+<layer number="2" name="Route2" color="1" fill="3" visible="no" active="no"/>
+<layer number="3" name="Route3" color="4" fill="3" visible="no" active="no"/>
+<layer number="4" name="Route4" color="1" fill="4" visible="no" active="no"/>
+<layer number="5" name="Route5" color="4" fill="4" visible="no" active="no"/>
+<layer number="6" name="Route6" color="1" fill="8" visible="no" active="no"/>
+<layer number="7" name="Route7" color="4" fill="8" visible="no" active="no"/>
+<layer number="8" name="Route8" color="1" fill="2" visible="no" active="no"/>
+<layer number="9" name="Route9" color="4" fill="2" visible="no" active="no"/>
+<layer number="10" name="Route10" color="1" fill="7" visible="no" active="no"/>
+<layer number="11" name="Route11" color="4" fill="7" visible="no" active="no"/>
+<layer number="12" name="Route12" color="1" fill="5" visible="no" active="no"/>
+<layer number="13" name="Route13" color="4" fill="5" visible="no" active="no"/>
+<layer number="14" name="Route14" color="1" fill="6" visible="no" active="no"/>
+<layer number="15" name="Route15" color="4" fill="6" visible="no" active="no"/>
+<layer number="16" name="Bottom" color="1" fill="1" visible="no" active="no"/>
+<layer number="17" name="Pads" color="2" fill="1" visible="no" active="no"/>
+<layer number="18" name="Vias" color="2" fill="1" visible="no" active="no"/>
+<layer number="19" name="Unrouted" color="6" fill="1" visible="no" active="no"/>
+<layer number="20" name="Dimension" color="15" fill="1" visible="no" active="no"/>
+<layer number="21" name="tPlace" color="7" fill="1" visible="no" active="no"/>
+<layer number="22" name="bPlace" color="7" fill="1" visible="no" active="no"/>
+<layer number="23" name="tOrigins" color="15" fill="1" visible="no" active="no"/>
+<layer number="24" name="bOrigins" color="15" fill="1" visible="no" active="no"/>
+<layer number="25" name="tNames" color="7" fill="1" visible="no" active="no"/>
+<layer number="26" name="bNames" color="7" fill="1" visible="no" active="no"/>
+<layer number="27" name="tValues" color="7" fill="1" visible="no" active="no"/>
+<layer number="28" name="bValues" color="7" fill="1" visible="no" active="no"/>
 <layer number="29" name="tStop" color="7" fill="3" visible="no" active="no"/>
 <layer number="30" name="bStop" color="7" fill="6" visible="no" active="no"/>
@@
 <layer number="35" name="tGlue" color="7" fill="4" visible="no" active="no"/>
 <layer number="36" name="bGlue" color="7" fill="5" visible="no" active="no"/>
-<layer number="37" name="tTest" color="7" fill="1" visible="yes" active="no"/>
-<layer number="38" name="bTest" color="7" fill="1" visible="yes" active="no"/>
+<layer number="37" name="tTest" color="7" fill="1" visible="no" active="no"/>
+<layer number="38" name="bTest" color="7" fill="1" visible="no" active="no"/>
 <layer number="39" name="tKeepout" color="4" fill="11" visible="no" active="no"/>
 <layer number="40" name="bKeepout" color="1" fill="11" visible="no" active="no"/>
@@
 <layer number="44" name="Drills" color="7" fill="1" visible="no" active="no"/>
 <layer number="45" name="Holes" color="7" fill="1" visible="no" active="no"/>
-<layer number="46" name="Milling" color="3" fill="1" visible="yes" active="no"/>
-<layer number="47" name="Measures" color="7" fill="1" visible="yes" active="no"/>
-<layer number="48" name="Document" color="7" fill="1" visible="yes" active="no"/>
-<layer number="49" name="Reference" color="7" fill="1" visible="yes" active="no"/>
-<layer number="51" name="tDocu" color="7" fill="1" visible="yes" active="no"/>
-<layer number="52" name="bDocu" color="7" fill="1" visible="yes" active="no"/>
+<layer number="46" name="Milling" color="3" fill="1" visible="no" active="no"/>
+<layer number="47" name="Measures" color="7" fill="1" visible="no" active="no"/>
+<layer number="48" name="Document" color="7" fill="1" visible="no" active="no"/>
+<layer number="49" name="Reference" color="7" fill="1" visible="no" active="no"/>
+<layer number="51" name="tDocu" color="7" fill="1" visible="no" active="no"/>
+<layer number="52" name="bDocu" color="7" fill="1" visible="no" active="no"/>
 <layer number="90" name="Modules" color="5" fill="1" visible="yes" active="yes"/>
 <layer number="91" name="Nets" color="2" fill="1" visible="yes" active="yes"/>
@@
 <net name="VIN" class="0">
 <segment>
-<pinref part="Q2" gate="G$1" pin="D"/>
-<wire x1="-99.06" y1="15.24" x2="-66.04" y2="15.24" width="0.1524" layer="91"/>
 <wire x1="-66.04" y1="15.24" x2="-53.34" y2="15.24" width="0.1524" layer="91"/>
 <wire x1="-53.34" y1="15.24" x2="-48.26" y2="15.24" width="0.1524" layer="91"/>
@@
 <wire x1="-30.48" y1="10.16" x2="-48.26" y2="15.24" width="0.1524" layer="91"/>
 <junction x="-48.26" y="15.24"/>
-<junction x="-66.04" y="15.24"/>
 <junction x="-53.34" y="15.24"/>
 <pinref part="C3" gate="G$1" pin="1"/>
@@
 <wire x1="-17.78" y1="15.24" x2="-20.32" y2="15.24" width="0.1524" layer="91"/>
 <junction x="-20.32" y="15.24"/>
-</segment>
-</net>
-<net name="N$2" class="0">
-<segment>
-<pinref part="Q1" gate="G$1" pin="S"/>
-<pinref part="Q2" gate="G$1" pin="S"/>
-<wire x1="-132.08" y1="15.24" x2="-114.3" y2="15.24" width="0.1524" layer="91"/>
-<wire x1="-114.3" y1="15.24" x2="-109.22" y2="15.24" width="0.1524" layer="91"/>
-<pinref part="R1" gate="G$1" pin="2"/>
-<wire x1="-114.3" y1="10.16" x2="-114.3" y2="15.24" width="0.1524" layer="91"/>
-<junction x="-114.3" y="15.24"/>
+<pinref part="Q2" gate="G$1" pin="D"/>
+<wire x1="-99.06" y1="15.24" x2="-66.04" y2="15.24" width="0.1524" layer="91"/>
+<junction x="-66.04" y="15.24"/>
 </segment>
 </net>
@@
 <wire x1="-106.68" y1="-17.78" x2="-106.68" y2="-25.4" width="0.1524" layer="91"/>
 <pinref part="J1" gate="G$1" pin="P2"/>
+</segment>
+</net>
+<net name="N$1" class="0">
+<segment>
+<pinref part="Q1" gate="G$1" pin="S"/>
+<pinref part="Q2" gate="G$1" pin="S"/>
+<wire x1="-132.08" y1="15.24" x2="-114.3" y2="15.24" width="0.1524" layer="91"/>
+<pinref part="R1" gate="G$1" pin="2"/>
+<wire x1="-114.3" y1="15.24" x2="-109.22" y2="15.24" width="0.1524" layer="91"/>
+<wire x1="-114.3" y1="10.16" x2="-114.3" y2="15.24" width="0.1524" layer="91"/>
+<junction x="-114.3" y="15.24"/>
 </segment>
 </net>
@@
 <part name="C4" library="rcl" deviceset="C-EU" device="C0603" value="2.2u"/>
 <part name="C5" library="rcl" deviceset="C-EU" device="C0603" value="18p"/>
-<part name="L3" library="rcl" deviceset="L-US" device="L1812" value="2.2u"/>
-<part name="L4" library="rcl" deviceset="L-US" device="L1812" value="2.2u"/>
+<part name="L3" library="rcl" deviceset="L-US" device="0603" value="2.2u"/>
+<part name="L4" library="rcl" deviceset="L-US" device="0603" value="2.2u"/>
 <part name="L1" library="rcl" deviceset="L-US" device="0603" value="47n"/>
 <part name="L2" library="rcl" deviceset="L-US" device="0603" value="47n"/>

Commit message: Routing of high-g IMU, regular IMU, firing circuits
1. Chose communication lines for all sensors and memory to the uC
2. Routed 100% the MPU9250
3. Routed 100% the high-g accelerometer
4. Routed 100% the breakwire circuits
5. Routed 75% of the firing circuits
Parts:
- removed R1: 10k, rcl:R-US_R0603
Connections:
- net MPU9250_SCL renamed IMU_SCL
- net MPU9250_SDA renamed IMU_SDA
- net N$20 renamed RTD_MISO
- net N$21 renamed RTD_MOSI
- removed net N$14: R1.2
- new net MEM_!CS: U1.PB14
- new net MEM_CS: U1.!CS
- new net MEM_MISO: U1.PA4, U1.SO/IO1
- new net MEM_MOSI: U1.PA3, U1.SI/IO0
- new net MEM_SCK: U1.PB13, U1.SCK
- new net RTD_!CS: U1.PA16
- new net RTD_SCK: U1.PA15
- net +3V3: no longer R1.2
- net GND: no longer R1.1
- net N$1: no longer R1.1, R1.2
- net N$3: no longer R1.2
- net N$4: no longer R1.1
- net N$5: no longer R1.1
- net PWR/PYRO+: no longer R1.1
- net SDA: no longer R1.1
Other:
- note added: "<-- LSB is 0"
- note added: "<-- LSB is 1"

Commit message: More routing and schematic changes
1. Finished 100% the schematic of all misc. connections that were going
to things, such as all comms, all LED indication pins, and all
enable/disable pins
2. Added FTDI FT232R for serial to USB connectivity
3. Routed the power line for the firing circuit from supercap
4. Routed LED indication
Parts:
- LED1, LED2, LED3, LED4, LED5: value (none) -> BLUE
- ON: value (none) -> RED
Connections:
- removed net FC1-1: J3.P4
- removed net FC1-2: J4.P2
- removed net FC1-3: J4.P4
- removed net N$12: J5.P4
- new net +5V: C1.2
- new net BW1_STATUS: J5.P2, U1.PB10
- new net BW2_STATUS: J5.P4, U1.PB11
- new net FC1_!CONT_EN: U1.PA0
- new net FC1_FIRE: U1.PA1
- new net FC2-: J3.P4, U1.PA26
- new net FC2_!CONT_EN: U1.PA2
- new net FC2_FIRE: U1.PA7
- new net FC3-: J4.P2, U1.PA30
- new net FC3_!CONT_EN: U1.PA8
- new net FC3_FIRE: U1.PA11
- new net FC4-: J4.P4, U1.PA31
- new net FC4_!CONT_EN: U1.PA14
- new net FC4_FIRE: U1.PA24
- new net ORD_!SHDN: U1.PA29
- new net USB_RX: U1.PB0
- new net USB_TX: U1.PB1
- net !SHDN: now also R4.1
- net FC1-: now also U1.PA25
- net GND: now also C1.1
- net N$10: no longer J5.P2
- net N$5: now also C2.1
- net UC_LED1: now also U1.PA17
- net UC_LED2: now also U1.PA18
- net UC_LED3: now also U1.PA19
- net UC_LED4: now also U1.PA20
- net UC_LED5: now also U1.PA23
Other:
- note added: "SPI2 Module"
- note added: "SPI3 Module"
- note added: "TWI0 Module"
- note added: "TWI1 Module"
- note added: "USART6 Module"
- note removed: "BW1_Status"
- note removed: "BW2_Status"
