File: GitHub Projects/CRAP Project/Flight Controller.brd (EAGLE design)
At the start: 40 x 90 mm, 114 parts, among them J1 2POS_SCREWTERM, J101 2POS_SCREWTERM, J2 4POS_SCREWTERM, J3 4POS_SCREWTERM, J4 4POS_SCREWTERM, J5 4POS_SCREWTERM, Q101 IPD042P03L3G, Q102 IPD042P03L3G

Commit message: Major changes
1. Cleaned up master level sheet
2. Changed MS5611 from SPI to I2C
3. Routed a lot
4. Changed MPU9250 power structure on top level (was broken)
5. Added serial communication lines to microcontroller
Parts:
- removed HIGH_G1:C1: 10u, rcl:C0805
- removed HIGH_G1:U1: HDLIS100DL, st-microelectronics:TFLGA16L
- removed IMU1:C1, IMU1:C3: 0.1u, rcl:C0603
- removed IMU1:C2: 10n, rcl:C0603
- removed IMU1:R2, IMU1:R3: 2.2K, rcl:R0603
- removed IMU1:U1: (no value), InvenSense:QFN-24
- added C601, C603: 0.1u, rcl:C0603
- added C602: 10n, rcl:C0603
- added C701: 100n, resistor:C0603
- added R602, R603: 2.2K, rcl:R0603
- added R701, R702: 2.2k, rcl:R0603
- added U601: (no value), InvenSense:QFN-24
- added U701: (no value), Measurement Specialties:MS5611
- C201: value 100n -> 10u; device resistor:C0603 -> rcl:C0805
- MEMORY1:U1: value (none) -> MT29F1G01
- U201: value (none) -> HDLIS100DL; device Measurement Specialties:MS5611 -> st-microelectronics:TFLGA16L
- moved C201 351.4 mm to (-119.0, -146.0)
- moved U201 346.7 mm to (-119.0, -138.0)
- moved C104 149.0 mm to (21.4, 72.0), flipped to the bottom, turned to 90 degrees
- moved R102 144.9 mm to (19.4, 68.6), flipped to the bottom, turned to 180 degrees
- moved R101 137.0 mm to (18.0, 72.0), flipped to the bottom, turned to 90 degrees
- moved C101 112.1 mm to (14.3, 85.8), turned to 270 degrees
- moved C103 106.6 mm to (9.31, 82.5)
- moved R106 106.4 mm to (12.1, 85.8), turned to 90 degrees
- moved L101 100.4 mm to (25.0, 85.0), turned to 270 degrees
- moved C102 100.0 mm to (9.75, 85.7), turned to 270 degrees
- moved Q102 95.5 mm to (10.1, 68.5), flipped to the bottom, turned to 270 degrees
- moved Q101 82.3 mm to (10.1, 78.0), flipped to the bottom, turned to 270 degrees
- moved U$101 38.3 mm to (18.0, 85.0)
- moved U1 17.0 mm to (20.0, 44.0)
- moved C305 9.00 mm to (24.0, 68.0)
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- renumbered BREAKWIRE1:C1 to C901, BREAKWIRE1:D1 to D901, BREAKWIRE1:R1 to R901, BREAKWIRE2:C1 to C1001, BREAKWIRE2:D1 to D1001, BREAKWIRE2:R1 to R1001, FIRING_CIRCUIT1:C1 to C1401, FIRING_CIRCUIT1:D1 to D1401, FIRING_CIRCUIT1:Q1 to Q1401, FIRING_CIRCUIT1:Q2 to Q1402, FIRING_CIRCUIT1:R1 to R1401, FIRING_CIRCUIT1:R2 to R1402, FIRING_CIRCUIT1:R3 to R1403, FIRING_CIRCUIT1:R4 to R1404, FIRING_CIRCUIT1:R5 to R1405, FIRING_CIRCUIT2:C1 to C1301, FIRING_CIRCUIT2:D1 to D1301, FIRING_CIRCUIT2:Q1 to Q1301, FIRING_CIRCUIT2:Q2 to Q1302, FIRING_CIRCUIT2:R1 to R1301, FIRING_CIRCUIT2:R2 to R1302, FIRING_CIRCUIT2:R3 to R1303, FIRING_CIRCUIT2:R4 to R1304, FIRING_CIRCUIT2:R5 to R1305, FIRING_CIRCUIT3:C1 to C1201, FIRING_CIRCUIT3:D1 to D1201, FIRING_CIRCUIT3:Q1 to Q1201, FIRING_CIRCUIT3:Q2 to Q1202, FIRING_CIRCUIT3:R1 to R1201, FIRING_CIRCUIT3:R2 to R1202, FIRING_CIRCUIT3:R3 to R1203, FIRING_CIRCUIT3:R4 to R1204, FIRING_CIRCUIT3:R5 to R1205, FIRING_CIRCUIT4:C1 to C1101, FIRING_CIRCUIT4:D1 to D1101, FIRING_CIRCUIT4:Q1 to Q1101, FIRING_CIRCUIT4:Q2 to Q1102, FIRING_CIRCUIT4:R1 to R1101, FIRING_CIRCUIT4:R2 to R1102, FIRING_CIRCUIT4:R3 to R1103, FIRING_CIRCUIT4:R4 to R1104, FIRING_CIRCUIT4:R5 to R1105, HIGH_G1:C2 to C202, HIGH_G1:C3 to C203
Connections:
- removed net BREAKWIRE2:BW_STAT/BW–: C1001.1
- removed net DCDC_REGULATOR:N$1: C101.1, C102.1, C103.1, Q102.2, R106.2, U$101.P13
- removed net IMU1:+3V3: IMU1:C1.1, IMU1:C2.1, IMU1:U1.1, IMU1:U1.10, IMU1:U1.8
- removed net IMU1:SCL: IMU1:R2.1, IMU1:U1.23
- removed net IMU1:SDA: IMU1:R3.1, IMU1:U1.24
- removed net MS5611_CS: U201.4, U201.5
- removed net MS5611_MISO: U201.6
- removed net MS5611_MOSI: U201.7
- removed net MS5611_SCLK: U201.8
- removed net XBEE900-1:XBEE_UART_IN: XB501.3
- removed net XBEE900-1:XBEE_UART_OUT: XB501.2
- new net DCDC_REGULATOR:VIN: C101.1, C102.1, C103.1, Q102.2, R106.2, U$101.P12, U$101.P13
- new net GPS_RX: U1.42
- new net GPS_TX: U1.43
- new net MPU9250_SCL: R602.1, U1.49, U601.23
- new net MPU9250_SDA: R603.1, U1.48, U601.24
- new net MS5611_SCL: R702.1, U1.39, U701.8
- new net MS5611_SDA: R701.1, U1.40, U701.7
- new net N$20: U1.8
- new net N$21: U1.17
- new net XBEE_RX: U1.21, XB501.3
- new net XBEE_TX: U1.51, XB501.2
- net +3V3: now also C601.1, C602.1, C603.1, C701.1, R602.2, R603.2, R701.2, R702.2, U201.P1, U201.P14, U201.P15, U601.1, U601.10, U601.13, U601.22, U601.8, U701.1, U701.2; no longer HIGH_G1:C1.1, HIGH_G1:U1.P1, HIGH_G1:U1.P14, HIGH_G1:U1.P15, IMU1:C3.1, IMU1:R2.2, IMU1:R3.2, IMU1:U1.13, IMU1:U1.22, U201.1
- net GND: now also C601.2, C602.2, C603.2, C701.2, U201.P10, U201.P12, U201.P13, U201.P16, U201.P5, U601.18, U601.20, U701.3, U701.4, U701.5; no longer HIGH_G1:C1.2, HIGH_G1:U1.P10, HIGH_G1:U1.P12, HIGH_G1:U1.P13, HIGH_G1:U1.P16, HIGH_G1:U1.P5, IMU1:C1.2, IMU1:C2.2, IMU1:C3.2, IMU1:U1.18, IMU1:U1.20, U201.2, U201.3
- net HIGH_G1:CS: now also U201.P8; no longer HIGH_G1:U1.P8
- net HIGH_G1:INT1: now also U201.P11; no longer HIGH_G1:U1.P11
- net HIGH_G1:INT2: now also U201.P9; no longer HIGH_G1:U1.P9
- net HIGH_G1:SCL/SPC: now also U201.P4; no longer HIGH_G1:U1.P4
- net HIGH_G1:SDA/SDI: now also U201.P6; no longer HIGH_G1:U1.P6
- net IMU1:INT: now also U601.12; no longer IMU1:U1.12
- net N$12: now also C1001.1
- net N$14: now also U601.9; no longer IMU1:U1.9
- net N$15: now also U201.P7; no longer HIGH_G1:U1.P7
Routing:
- net +3V3: track 0.00 -> 105.4 mm, vias 0 -> 4
- net DCDC_REGULATOR:VIN: track 0.00 -> 35.6 mm, vias 0 -> 1
- net DCDC_REGULATOR:N$6: track 0.00 -> 26.6 mm
- net DCDC_REGULATOR:N$2: track 0.00 -> 19.9 mm
- net VCC_IN: track 0.00 -> 19.2 mm
- net N$3: track 0.00 -> 13.0 mm, vias 0 -> 1
- net MPU9250_SDA: track 0.00 -> 12.1 mm, vias 0 -> 1
- net DCDC_REGULATOR:N$4: track 0.00 -> 11.2 mm
- net N$1: track 0.00 -> 11.0 mm
- net N$2: track 0.00 -> 9.74 mm
- net MPU9250_SCL: track 0.00 -> 8.85 mm, vias 0 -> 1
- net DCDC_REGULATOR:N$11: track 0.00 -> 8.65 mm
- net N$4: track 0.00 -> 7.98 mm
- net MS5611_SDA: track 0.00 -> 7.95 mm
- net DCDC_REGULATOR:N$5: track 0.00 -> 7.16 mm
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
Commit message: Routed more, added GPS
1. Added Antenova library
2. Added our GPS to the Antenova library
3. Placed GPS, which caused our power system to move, also increased
board height by 5mm due to expected space constraints
4. Moved our power system close to the Xbee
5. Placed a MOSFET for the separation circuit
Parts:
- added C801, C802, C803: 22p, rcl:C0603
- added C804: 2.2u, rcl:C0603
- added C805: 18p, rcl:C0603
- added L801, L802: 47n, rcl:L1812
- added L803, L804: 2.2u, rcl:L1812
- added U$801: (no value), Antenova:M10478-A3
- moved C102 52.3 mm to (15.8, 33.7)
- moved C101 52.3 mm to (20.3, 33.8)
- moved C103 52.3 mm to (15.3, 30.5)
- moved U$101 52.3 mm to (24.0, 33.0)
- moved R106 52.3 mm to (18.1, 33.8)
- moved L101 46.4 mm to (31.0, 39.0), turned to 0 degrees
- moved Q1402 45.2 mm to (27.0, 48.0), flipped to the bottom, turned to 90 degrees
- moved C104 8.42 mm to (13.0, 71.4), turned to 0 degrees
- moved R101 5.39 mm to (13.0, 74.0), turned to 0 degrees
- moved Q101 3.14 mm to (7.05, 77.1), turned to 180 degrees
- moved C305 3.00 mm to (24.0, 71.0)
- moved C601 3.00 mm to (16.2, 60.3)
- moved C602 3.00 mm to (13.6, 60.4)
- moved C603 3.00 mm to (20.9, 62.8)
- moved C701 3.00 mm to (28.0, 60.1)
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Connections:
- new net GPS1:+3V3: C803.2, C804.2, U$801.8
- new net GPS1:GND: C801.2, C802.2, C803.1, C804.1, L803.1, L804.1, U$801.1, U$801.15, U$801.16, U$801.17, U$801.19, U$801.2, U$801.22, U$801.23, U$801.24, U$801.25, U$801.27, U$801.28, U$801.3, U$801.5, U$801.7, U$801.9
- new net GPS1:GPS_RX: L801.2
- new net GPS1:GPS_TX: L802.2
- new net GPS1:N$1: C805.1, L803.2, U$801.4
- new net GPS1:N$2: C802.1, L801.1, U$801.21
- new net GPS1:N$3: C801.1, L802.1, U$801.20
- new net GPS1:N$4: C805.2, L804.2, U$801.6
Routing:
- net +3V3: track 105.4 -> 75.0 mm
- net DCDC_REGULATOR:VIN: track 35.6 -> 18.9 mm
- net VCC_IN: track 19.2 -> 29.9 mm
- net DCDC_REGULATOR:N$6: track 26.6 -> 35.8 mm
- net DCDC_REGULATOR:N$5: track 7.16 -> 13.2 mm
- net FC1-: track 0.00 -> 4.80 mm
- net DCDC_REGULATOR:N$2: track 19.9 -> 22.8 mm
- net DCDC_REGULATOR:N$4: track 11.2 -> 9.78 mm
Other:
- board size 40 x 90 mm -> 40 x 93 mm
